File: WS2812.sch (KiCad schematic (older format))
At the start: 10 parts, among them P6 ws2812, Q1 S9013, Q2 S9013, Q3 S9013

Commit message: Draft for revision 1.1
Parts:
- removed Q1, Q2: S9013, Housings_SOT-23_SOT-143_TSOT-6:SOT-23_Handsoldering, symbol Q_NPN_BEC-RESCUE-RPi_Hat
- removed R17: 1k, Resistors_SMD:R_0603_HandSoldering, symbol R
- removed R18: 10k, Resistors_SMD:R_0603_HandSoldering, symbol R
- added C20: 1u, Capacitors_SMD:C_0603_HandSoldering, symbol C_Small
- added F2: F_Small, Fuse_Holders_and_Fuses:Fuse_SMD1206_HandSoldering, symbol F_Small
- renumbered Q3 to Q1, R19 to R30, R20 to R31, R21 to R32
Connections:
- wire segments 27 -> 25
Changed lines of the file:
@@
 EESchema Schematic File Version 2
-LIBS:RPi_Hat-rescue
 LIBS:power
 LIBS:device
@@
 LIBS:adc-dac
 LIBS:memory
-LIBS:xilinx
-LIBS:special
 LIBS:microcontrollers
 LIBS:dsp
@@
 LIBS:valves
 LIBS:MP1496
+LIBS:LOGIC-TXS0108EPWR_TSSOP20_
+LIBS:RPi_Hat
 LIBS:RPi_Hat-cache
 EELAYER 25 0
@@
 $Descr A4 11693 8268
 encoding utf-8
-Sheet 3 3
+Sheet 2 3
 Title ""
 Date ""
@@
 $EndDescr
 $Comp
-L R R19
+L R R30
 U 1 1 554A668D
 P 5700 3100
-F 0 "R19" V 5780 3100 50  0000 C CNN
+F 0 "R30" V 5780 3100 50  0000 C CNN
 F 1 "1.5k" V 5700 3100 50  0000 C CNN
 F 2 "Resistors_SMD:R_0603_HandSoldering" V 5630 3100 30  0001 C CNN
@@
 $EndComp
 $Comp
-L R R20
+L R R31
 U 1 1 554A6694
 P 6050 3100
-F 0 "R20" V 6130 3100 50  0000 C CNN
+F 0 "R31" V 6130 3100 50  0000 C CNN
 F 1 "4.7k" V 6050 3100 50  0000 C CNN
 F 2 "Resistors_SMD:R_0603_HandSoldering" V 5980 3100 30  0001 C CNN
@@
 $EndComp
 $Comp
-L R R21
+L R R32
 U 1 1 554A669C
 P 6050 3950
-F 0 "R21" V 6130 3950 50  0000 C CNN
+F 0 "R32" V 6130 3950 50  0000 C CNN
 F 1 "1.1k" V 6050 3950 50  0000 C CNN
 F 2 "Resistors_SMD:R_0603_HandSoldering" V 5980 3950 30  0001 C CNN
@@
 $EndComp
 $Comp
-L GND #PWR25
+L GND #PWR024
 U 1 1 554A66A3
 P 6250 4150
-F 0 "#PWR25" H 6250 3900 50  0001 C CNN
+F 0 "#PWR024" H 6250 3900 50  0001 C CNN
 F 1 "GND" H 6250 4000 50  0000 C CNN
 F 2 "" H 6250 4150 60  0000 C CNN
@@
 $EndComp
 $Comp
-L GND #PWR22
+L GND #PWR025
 U 1 1 554A66B1
-P 3650 3050
-F 0 "#PWR22" H 3650 2800 50  0001 C CNN
-F 1 "GND" H 3650 2900 50  0000 C CNN
-F 2 "" H 3650 3050 60  0000 C CNN
-F 3 "" H 3650 3050 60  0000 C CNN
-	1    3650 3050
+P 3650 3250
+F 0 "#PWR025" H 3650 3000 50  0001 C CNN
+F 1 "GND" H 3650 3100 50  0000 C CNN
+F 2 "" H 3650 3250 60  0000 C CNN
+F 3 "" H 3650 3250 60  0000 C CNN
+	1    3650 3250
 	1    0    0    -1
 $EndComp
 $Comp
-L Q_NPN_BEC-RESCUE-RPi_Hat Q3
+L Q_NPN_BEC-RESCUE-RPi_Hat Q1
 U 1 1 554A66B7
 P 5800 3600
-F 0 "Q3" H 6100 3650 50  0000 R CNN
+F 0 "Q1" H 6100 3650 50  0000 R CNN
 F 1 "S9013" H 6400 3550 50  0000 R CNN
 F 2 "Housings_SOT-23_SOT-143_TSOT-6:SOT-23_Handsoldering" H 6000 3700 29  0001 C CNN
@@
 	1    5800 3600
 	-1   0    0    -1
-$EndComp
-$Comp
-L Q_NPN_BEC-RESCUE-RPi_Hat Q2
-U 1 1 554A66BE
-P 5000 3350
-F 0 "Q2" H 5300 3400 50  0000 R CNN
-F 1 "S9013" H 5600 3300 50  0000 R CNN
-F 2 "Housings_SOT-23_SOT-143_TSOT-6:SOT-23_Handsoldering" H 5200 3450 29  0001 C CNN
-F 3 "" H 5000 3350 60  0000 C CNN
-	1    5000 3350
-	-1   0    0    -1
-$EndComp
-$Comp
-L GND #PWR24
-U 1 1 554A66C5
-P 4900 3650
-F 0 "#PWR24" H 4900 3400 50  0001 C CNN
-F 1 "GND" H 4900 3500 50  0000 C CNN
-F 2 "" H 4900 3650 60  0000 C CNN
-F 3 "" H 4900 3650 60  0000 C CNN
-	1    4900 3650
-	1    0    0    -1
-$EndComp
-$Comp
-L R R18
-U 1 1 554A66CB
-P 4900 2900
-F 0 "R18" V 4980 2900 50  0000 C CNN
-F 1 "10k" V 4900 2900 50  0000 C CNN
-F 2 "Resistors_SMD:R_0603_HandSoldering" V 4830 2900 30  0001 C CNN
-F 3 "" H 4900 2900 30  0000 C CNN
-	1    4900 2900
-	-1   0    0    1
-$EndComp
-$Comp
-L +5V #PWR23
-U 1 1 554A66D2
-P 4900 2450
-F 0 "#PWR23" H 4900 2300 50  0001 C CNN
-F 1 "+5V" H 4900 2590 50  0000 C CNN
-F 2 "" H 4900 2450 60  0000 C CNN
-F 3 "" H 4900 2450 60  0000 C CNN
-	1    4900 2450
-	1    0    0    -1
-$EndComp
-$Comp
-L Q_NPN_BEC-RESCUE-RPi_Hat Q1
-U 1 1 554A66D8
-P 4500 3100
-F 0 "Q1" H 4800 3150 50  0000 R CNN
-F 1 "S9013" H 5100 3050 50  0000 R CNN
-F 2 "Housings_SOT-23_SOT-143_TSOT-6:SOT-23_Handsoldering" H 4700 3200 29  0001 C CNN
-F 3 "" H 4500 3100 60  0000 C CNN
-	1    4500 3100
-	-1   0    0    -1
-$EndComp
-$Comp
-L R R17
-U 1 1 554A66DF
-P 4400 2650
-F 0 "R17" V 4480 2650 50  0000 C CNN
-F 1 "1k" V 4400 2650 50  0000 C CNN
-F 2 "Resistors_SMD:R_0603_HandSoldering" V 4330 2650 30  0001 C CNN
-F 3 "" H 4400 2650 30  0000 C CNN
-	1    4400 2650
-	-1   0    0    1
 $EndComp
 $Comp
@@
 $EndComp
 $Comp
-L +5V #PWR21
+L +5V #PWR026
 U 1 1 554A66ED
-P 3650 2700
-F 0 "#PWR21" H 3650 2550 50  0001 C CNN
-F 1 "+5V" H 3650 2840 50  0000 C CNN
-F 2 "" H 3650 2700 60  0000 C CNN
-F 3 "" H 3650 2700 60  0000 C CNN
-	1    3650 2700
+P 3650 2400
+F 0 "#PWR026" H 3650 2250 50  0001 C CNN
+F 1 "+5V" H 3650 2540 50  0000 C CNN
+F 2 "" H 3650 2400 60  0000 C CNN
+F 3 "" H 3650 2400 60  0000 C CNN
+	1    3650 2400
 	1    0    0    -1
 $EndComp
@@
 Connection ~ 5700 3350
 Wire Wire Line
-	3650 3050 3650 2950
+	3650 2950 3650 3250
 Wire Wire Line
 	3650 2950 3600 2950
 Wire Wire Line
-	4900 3550 4900 3650
-Wire Wire Line
-	5200 3350 5700 3350
-Wire Wire Line
-	4900 3050 4900 3150
-Wire Wire Line
-	4900 2450 4900 2750
-Wire Wire Line
-	4700 3100 4900 3100
-Connection ~ 4900 3100
-Wire Wire Line
-	4400 2500 4900 2500
-Connection ~ 4900 2500
-Wire Wire Line
-	4400 2800 4400 2900
-Wire Wire Line
-	4400 3300 4400 3600
-Wire Wire Line
-	4400 3600 4900 3600
-Connection ~ 4900 3600
-Wire Wire Line
-	3600 2850 4400 2850
-Connection ~ 4400 2850
-Wire Wire Line
-	3650 2700 3650 2750
+	3650 2650 3650 2750
 Wire Wire Line
 	3650 2750 3600 2750
@@
 Wire Wire Line
 	5700 4500 6000 4500
+$Comp
+L F_Small F2
+U 1 1 56C10670
+P 3650 2550
+F 0 "F2" H 3610 2610 50  0000 L CNN
+F 1 "F_Small" H 3530 2490 50  0000 L CNN
+F 2 "Fuse_Holders_and_Fuses:Fuse_SMD1206_HandSoldering" H 3650 2550 50  0001 C CNN
+F 3 "" H 3650 2550 50  0000 C CNN
+	1    3650 2550
+	0    1    1    0
+$EndComp
+Wire Wire Line
+	3650 2400 3650 2450
+Wire Wire Line
+	4650 3350 5700 3350
+Wire Wire Line
+	4650 3350 4650 2850
+Wire Wire Line
+	4650 2850 3600 2850
+$Comp
+L C_Small C20
+U 1 1 56C10EB7
+P 4000 3050
+F 0 "C20" H 4010 3120 50  0000 L CNN
+F 1 "1u" H 4010 2970 50  0000 L CNN
+F 2 "Capacitors_SMD:C_0603_HandSoldering" H 4000 3050 60  0001 C CNN
+F 3 "" H 4000 3050 60  0000 C CNN
+	1    4000 3050
+	-1   0    0    1
+$EndComp
+Wire Wire Line
+	4000 3150 4000 3200
+Wire Wire Line
+	4000 3200 3650 3200
+Connection ~ 3650 3200
+Wire Wire Line
+	4000 2950 4000 2700
+Wire Wire Line
+	4000 2700 3650 2700
+Connection ~ 3650 2700
 $EndSCHEMATC
